File: hardware/flight_stick.kicad_pcb (KiCad board)
At the start: 4 copper layers, 76 x 51.5 mm, 60 parts, among them J1 Conn_01x04_Male, J10 USB_C_Receptacle_USB2.0, J12 Load Cell 2, J2 Conn_02x05_Odd_Even, J3 Conn_01x04_Male, J4 Load Cell 3, J6 Load Cell 1, J9 Conn_ST_STDC14, SW1 KMR223G LFG, U2 AT24CS01-MAHM, U3 ADS131M03IRUKx, U4 STM32F103CBU6, U5 USBLC6-2SC6, U6 TCAN3403, U7 LT1962-3.3, U8 TPS62177DQC, Y1 8M

Commit message: adding overdue changes
Routing:
- added copper zone on B.Cu, net GND
- added copper zone on F.Cu, net GND
- added copper zone on B.Cu, net GNDA
- added copper zone on F.Cu, net GNDA
Changed lines of the file:
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@@
 		(layer "Cmts.User")
 		(pts
+			(xy 91.819013 38.383891) (xy 86.56 89.92)
+		)
+		(height 42.500987)
+		(orientation 1)
+		(format
+			(prefix "")
+			(suffix "")
+			(units 3)
+			(units_format 1)
+			(precision 4)
+		)
+		(style
+			(thickness 0.2)
+			(arrow_length 1.27)
+			(text_position_mode 2)
+			(arrow_direction outward)
+			(extension_height 0.58642)
+			(extension_offset 0.5)
+			(keep_text_aligned yes)
+		)
+		(gr_text "51.5361 mm"
+			(at 131.96 62.92 90)
+			(layer "Cmts.User")
+			(effects
+				(font
+					(size 1.5 1.5)
+					(thickness 0.3)
+				)
+			)
+		)
+	)
+	(dimension
+		(type orthogonal)
+		(layer "Cmts.User")
+		(pts
 			(xy 73.819013 77.383891) (xy 105.819013 44.383891)
 		)
@@
 	)
 	(zone
-		(net 57)
-		(net_name "+3.3VA")
-		(layer "In1.Cu")
+		(net 75)
+		(net_name "GNDA")
+		(layers "F.Cu" "B.Cu" "In2.Cu")
 		(hatch edge 0.5)
-		(priority 3)
 		(connect_pads
 			(clearance 0.2)
@@
 		(polygon
 			(pts
-				(xy 68.819013 58.883891) (xy 62.319013 56.383891) (xy 57.819013 61.383891) (xy 49.819013 59.883891)
-				(xy 41.819013 59.883891) (xy 40.819013 58.883891) (xy 32.819013 58.883891) (xy 32.819013 34.883891)
-				(xy 58.319013 35.383891) (xy 61.319013 44.883891) (xy 67.319013 52.883891) (xy 77.819013 53.883891)
-				(xy 77.319013 59.383891) (xy 71.319013 59.383891)
+				(xy 54.819013 60.883891) (xy 49.819013 59.883891) (xy 41.819013 59.883891) (xy 40.819013 58.883891)
+				(xy 33.819013 58.883891) (xy 33.819013 35.883891) (xy 57.319013 36.383891) (xy 60.319013 45.383891)
+				(xy 67.319013 52.883891) (xy 78.319013 53.883891) (xy 77.819013 60.383891) (xy 64.819013 60.383891)
+				(xy 62.319013 58.383891) (xy 61.319013 58.383891) (xy 57.819013 61.383891)
 			)
 		)
 	)
 	(zone
-		(net 1)
-		(net_name "+3.3V")
-		(layer "In1.Cu")
+		(net 2)
+		(net_name "GND")
+		(layers "F.Cu" "B.Cu" "In2.Cu")
 		(hatch edge 0.5)
-		(priority 2)
+		(priority 1)
 		(connect_pads
 			(clearance 0.2)
@@
 		(polygon
 			(pts
-				(xy 40.819013 59.383891) (xy 41.819013 60.383891) (xy 49.819013 60.383891) (xy 57.819013 61.883891)
-				(xy 62.319013 56.883891) (xy 70.819013 59.883891) (xy 77.819013 59.883891) (xy 78.319013 53.883891)
-				(xy 84.819013 50.883891) (xy 89.319013 43.883891) (xy 90.819013 34.383891) (xy 116.319013 34.383891)
-				(xy 115.819013 69.383891) (xy 92.319013 93.883891) (xy 56.819013 93.883891) (xy 31.49498 69.066339)
-				(xy 31.819013 59.383891)
+				(xy 41.021544 59.383891) (xy 41.819013 60.283891) (xy 50.019013 60.283891) (xy 54.819013 61.383891)
+				(xy 57.819013 61.883891) (xy 61.319013 58.883891) (xy 62.319013 58.883891) (xy 64.819013 60.883891)
+				(xy 78.319013 60.883891) (xy 78.819013 53.883891) (xy 85.019013 50.783891) (xy 89.519013 43.783891)
+				(xy 91.019013 36.283891) (xy 114.519013 36.283891) (xy 114.019013 68.783891) (xy 91.519013 91.783891)
+				(xy 57.519013 92.283891) (xy 33.519013 68.783891) (xy 33.690964 59.383891)
 			)
 		)
 	)
 	(zone
-		(net 75)
-		(net_name "GNDA")
-		(layer "In2.Cu")
+		(net 57)
+		(net_name "+3.3VA")
+		(layer "In1.Cu")
 		(hatch edge 0.5)
+		(priority 3)
 		(connect_pads
 			(clearance 0.2)
@@
 		(polygon
 			(pts
-				(xy 54.819013 60.883891) (xy 49.819013 59.883891) (xy 41.819013 59.883891) (xy 40.819013 58.883891)
-				(xy 33.819013 58.883891) (xy 33.819013 35.883891) (xy 57.319013 36.383891) (xy 60.319013 45.383891)
-				(xy 67.319013 52.883891) (xy 78.319013 53.883891) (xy 77.819013 60.383891) (xy 64.819013 60.383891)
-				(xy 62.319013 58.383891) (xy 61.319013 58.383891) (xy 57.819013 61.383891)
+				(xy 68.819013 58.883891) (xy 62.319013 56.383891) (xy 57.819013 61.383891) (xy 49.819013 59.883891)
+				(xy 41.819013 59.883891) (xy 40.819013 58.883891) (xy 32.819013 58.883891) (xy 32.819013 34.883891)
+				(xy 58.319013 35.383891) (xy 61.319013 44.883891) (xy 67.319013 52.883891) (xy 77.819013 53.883891)
+				(xy 77.319013 59.383891) (xy 71.319013 59.383891)
 			)
 		)
 	)
 	(zone
-		(net 2)
-		(net_name "GND")
-		(layer "In2.Cu")
+		(net 1)
+		(net_name "+3.3V")
+		(layer "In1.Cu")
 		(hatch edge 0.5)
-		(priority 1)
+		(priority 2)
 		(connect_pads
 			(clearance 0.2)
@@
 		(polygon
 			(pts
-				(xy 41.021544 59.383891) (xy 41.819013 60.283891) (xy 50.019013 60.283891) (xy 54.819013 61.383891)
-				(xy 57.819013 61.883891) (xy 61.319013 58.883891) (xy 62.319013 58.883891) (xy 64.819013 60.883891)
-				(xy 78.319013 60.883891) (xy 78.819013 53.883891) (xy 85.019013 50.783891) (xy 89.519013 43.783891)
-				(xy 91.019013 36.283891) (xy 114.519013 36.283891) (xy 114.019013 68.783891) (xy 91.519013 91.783891)
-				(xy 57.519013 92.283891) (xy 33.519013 68.783891) (xy 33.690964 59.383891)
+				(xy 40.819013 59.383891) (xy 41.819013 60.383891) (xy 49.819013 60.383891) (xy 57.819013 61.883891)
+				(xy 62.319013 56.883891) (xy 70.819013 59.883891) (xy 77.819013 59.883891) (xy 78.319013 53.883891)
+				(xy 84.819013 50.883891) (xy 89.319013 43.883891) (xy 90.819013 34.383891) (xy 116.319013 34.383891)
+				(xy 115.819013 69.383891) (xy 92.319013 93.883891) (xy 56.819013 93.883891) (xy 31.49498 69.066339)
+				(xy 31.819013 59.383891)
 			)
 		)
