File: hardware/flight_stick.kicad_sch (KiCad schematic)
At the start: 22 parts, among them J10 USB_C_Receptacle_USB2.0, J2 Conn_02x05_Odd_Even, J9 Conn_ST_STDC14, SW1 KMR223G LFG, U2 AT24CS01-MAHM, U4 STM32F103CBU6, U5 USBLC6-2SC6, Y1 8M

Commit message: adding overdue changes
Changed lines of the file:
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@@
 		(on_board yes)
 		(dnp no)
-		(fields_autoplaced yes)
 		(property "Reference" "U4"
-			(at 94.9041 177.8 0)
+			(at 94.742 179.578 0)
 			(effects
 				(font
@@
 		)
 		(property "Value" "STM32F103CBU6"
-			(at 94.9041 180.34 0)
+			(at 94.742 182.118 0)
 			(effects
 				(font
